File: hw/ESPDali.kicad_sch (KiCad schematic)
At the start: 52 parts, among them J1 2pin 3.5mm terminal block, J2 2pin 3.5mm terminal block, J3 2.54mm pin header, Q1 BCX56-16, Q2 SMBT2222A, Q3 BCX56-16, SW1 SW_Push, SW2 SW_Push, U1 LM27313XMF, U2 TLP185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

Commit message: Footprint fixes to PCB
Parts:
- removed C10, C11: 1n, Capacitor_SMD:C_0603_1608Metric, symbol Device:C
- removed D2: MB1S, ESPDali:MB1S, symbol Device:D_Bridge_+AA-
- removed R15, R16: 470R, Resistor_SMD:R_0603_1608Metric, symbol Device:R
- removed SW1, SW2: SW_Push, Button_Switch_SMD:SW_Push_SPST_NO_Alps_SKRK, symbol Switch:SW_Push
- removed U3: MCP1804x-3302xDB, Package_TO_SOT_SMD:SOT-223-3_TabPin2, symbol Regulator_Linear:MCP1804x-3302xDB
- added D2: MB1S, ESPDali:MB1S, symbol Device:D_Bridge_+-AA
- added U3: SPX2920M3-3.3_SOT223, Package_TO_SOT_SMD:SOT-223-3_TabPin2, symbol Regulator_Linear:SPX2920M3-3.3_SOT223
- J3: footprint Connector_PinHeader_2.54mm:PinHeader_1x03_P2.54mm_Vertical -> Connector_PinHeader_2.54mm:PinHeader_1x05_P2.54mm_Vertical; symbol Connector_Generic:Conn_01x03 -> Connector_Generic:Conn_01x05
- R2: value 100k -> 330
- R6: value 13.3k -> 13k
Connections:
- net +3V3: now also U3.3 (VO)
- net BOOT: now also J3.4 (Pin_4)
- net GND: now also U3.2 (GND)
- net GNDPWR: now also D2.2 (-)
- net LED: now also U5.36 (IO22); no longer U5.24 (IO2)
- net VIN: now also U3.1 (VI)
- net at C4.1, F1.2, J2.1 (Pin_1): now also D2.4
- net at C4.2, J2.2 (Pin_2), R10.1: now also D2.3
- net at R8.2, R9.2: now also D2.1 (+)
- net RESET renamed EN
- net EN: now also J3.5 (Pin_5)
Other:
- note added: "18V Boost"
- note added: "3.3V >250mA LDO"
- note added: "5V, 1.5A"
- note added: "C4 optionally 100p shunts possible high frequencies on the line."
- note added: "DALI Bus Driver"
- note added: "EPS32 consumes in-rush >250mA on average 50 mA"
- note added: "External supply 4-18V"
- note added: "Inverted signal!"
- note removed: "16V Boost"
- note removed: "3.3V LDO"
- note removed: "C4 optionally 100p shunts possible AC on the line."
- note removed: "EPS32 consumes max 50 mA"
- note removed: "External supply 4-14V"

Commit message: Update to KiCAD 8
Parts:
- C4: now not fitted
- U3: value SPX2920M3-3.3_SOT223 -> MCP1703A-330
Connections:
- net DALI_RX: now also U5.27 (IO16); no longer U5.23 (IO15)
Other:
- note added: "LT1129IST-3.3 LT1963EST-3.3 MCP1703A-330 SPX2920M3-3.3_SOT223"
- note added: "Populate C4 to shunt high frequencies on the line."
- note added: "Pretty much any optocoupler works - TLP185 - TCLT1000 - PC357N4"
- note removed: "C4 optionally 100p shunts possible high frequencies on the line."
- note removed: "Pretty much any optocoupler works - TCLT1000 - PC357N4"
- moved on the sheet: C7, C8, C9, D5, D6, R13, R14, R17, R18, U5
